File: PROJECT_ENTERPRISE_1.kicad_sch (KiCad schematic)
At the start: 63 parts, among them J1 USB_C_Receptacle_USB2.0_16P, J2 Battery Input, J3 Battery Input, J4 Battery Input, J5 Battery Input, Q2 IRF7343PBF, Q3 IRF7343PBF, Q4 IRF7343PBF, Q5 IRF7343PBF, SW1 RESET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

Commit message: added the code
Parts:
- added R34: 220 2Watt, Resistor_SMD:R_1206_3216Metric_Pad1.30x1.75mm_HandSolder, symbol Device:R
Connections:
- net at J5.2 (Pin_2), Q5.7 (D1), Q5.8 (D1)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: now also R34.2
- net at J5.1 (Pin_1), Q5.3 (S2): now also R34.1
Changed lines of the file:
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@@
 	)
 	(junction
+		(at 72.39 134.62)
+		(diameter 0)
+		(color 0 0 0 0)
+	)
+	(junction
 		(at 48.26 69.85)
 		(diameter 0)
@@
 	)
 	(junction
+		(at 72.39 142.24)
+		(diameter 0)
+		(color 0 0 0 0)
+	)
+	(junction
 		(at 29.21 123.19)
 		(diameter 0)
@@
 	(wire
 		(pts
-			(xy 72.39 138.43) (xy 72.39 147.32)
+			(xy 72.39 138.43) (xy 72.39 142.24)
 		)
 		(stroke
@@
 	(wire
 		(pts
+			(xy 66.04 134.62) (xy 72.39 134.62)
+		)
+		(stroke
+			(width 0)
+			(type default)
+		)
+	)
+	(wire
+		(pts
 			(xy 81.28 147.32) (xy 82.55 147.32)
 		)
@@
 	(wire
 		(pts
+			(xy 72.39 142.24) (xy 72.39 147.32)
+		)
+		(stroke
+			(width 0)
+			(type default)
+		)
+	)
+	(wire
+		(pts
 			(xy 72.39 85.09) (xy 72.39 111.76)
 		)
@@
 	(wire
 		(pts
+			(xy 72.39 134.62) (xy 72.39 135.89)
+		)
+		(stroke
+			(width 0)
+			(type default)
+		)
+	)
+	(wire
+		(pts
 			(xy 16.51 68.58) (xy 20.32 68.58)
 		)
@@
 	(wire
 		(pts
+			(xy 66.04 142.24) (xy 72.39 142.24)
+		)
+		(stroke
+			(width 0)
+			(type default)
+		)
+	)
+	(wire
+		(pts
 			(xy 184.15 161.29) (xy 193.04 161.29)
 		)
@@
 	(wire
 		(pts
-			(xy 72.39 125.73) (xy 72.39 135.89)
+			(xy 72.39 125.73) (xy 72.39 134.62)
 		)
 		(stroke
@@
 					(unit 1)
 				)
+			)
+		)
+	)
+	(symbol
+		(lib_id "Device:R")
+		(at 66.04 138.43 0)
+		(unit 1)
+		(body_style 1)
+		(exclude_from_sim no)
+		(in_bom yes)
+		(on_board yes)
+		(in_pos_files yes)
+		(dnp no)
+		(property "Reference" "R34"
+			(at 66.04 138.43 90)
+			(show_name no)
+			(do_not_autoplace no)
+			(effects
+				(font
+					(size 1.27 1.27)
+				)
+			)
+		)
+		(property "Value" "220 2Watt"
+			(at 59.436 138.43 0)
+			(show_name no)
+			(do_not_autoplace no)
+			(effects
+				(font
+					(size 1.27 1.27)
+				)
+			)
+		)
+		(property "Footprint" "Resistor_SMD:R_1206_3216Metric_Pad1.30x1.75mm_HandSolder"
+			(at 64.262 138.43 90)
+			(hide yes)
+			(show_name no)
+			(do_not_autoplace no)
+			(effects
+				(font
+					(size 1.27 1.27)
+				)
+			)
+		)
+		(property "Datasheet" ""
+			(at 66.04 138.43 0)
+			(hide yes)
+			(show_name no)
+			(do_not_autoplace no)
+			(effects
+				(font
+					(size 1.27 1.27)
+				)
+			)
+		)
+		(property "Description" "Resistor"
+			(at 66.04 138.43 0)
+			(hide yes)
+			(show_name no)
+			(do_not_autoplace no)
+			(effects
+				(font
+					(size 1.27 1.27)
+				)
+			)
+		)
+		(pin "1"
+		)
+		(pin "2"
+		)
+		(instances
+			(project "PROJECT_ENTERPRISE_1"
+				(path "/8e52210a-ef94-47f7-a0af-9c2bdf0282f0"
+					(reference "R34")
+					(unit 1)
+				)

Commit message: transistor
Parts:
- removed R16: 100K, Resistor_SMD:R_1206_3216Metric_Pad1.30x1.75mm_HandSolder, symbol Device:R
- removed R34: 220 2Watt, Resistor_SMD:R_1206_3216Metric_Pad1.30x1.75mm_HandSolder, symbol Device:R
- added Q1: BC547, Package_TO_SOT_THT:TO-92_Inline, symbol Transistor_BJT:BC547
- added R13: 2 Ohm, Resistor_SMD:R_1206_3216Metric_Pad1.30x1.75mm_HandSolder, symbol Device:R
- added R35: 10k, Resistor_SMD:R_1206_3216Metric_Pad1.30x1.75mm_HandSolder, symbol Device:R
- added R36: 1K, Resistor_SMD:R_1206_3216Metric_Pad1.30x1.75mm_HandSolder, symbol Device:R
- R24: value 100 -> 1K
Connections:
- net +5V: no longer R11.2
- net A_Sense1: now also Q5.1 (S1), R13.2, R36.1
- net GND: now also Q1.1 (C), R13.1, R35.1; no longer D5.2 (A), Q5.1 (S1)
- net at Q5.2 (G1), R24.2: now also Q1.3 (E), R35.2
- net at J5.2 (Pin_2), Q5.7 (D1), Q5.8 (D1): no longer R8.1
- new net: Q1.2 (B), R36.2
Other:
- moved on the sheet: D5, D6, R11, R15, R24, R8
