File: PROJECT_1_V2.kicad_pcb (KiCad board)
At the start: 4 copper layers, 69 x 52.5 mm, 125 parts, among them J1 Battery Input, J2 Battery Input, J3 Battery Input, J4 Battery Input, J5 USB_C_Receptacle_USB2.0_16P, Q10 DMG9926UDM, Q7 DMG9926UDM, Q8 DMG9926UDM, Q9 DMG9926UDM, SW1 RESET, SW2 BOOT_LOADER, U1 TP4056, U10 DW01A, U11 TP4056-42-ESOP8, U12 DW01A, U2 Nokia_5110_LCD, U3 LM2576T-3.3, U4 RP2040, U5 W25Q128JVS, U6 DW01A, U7 TP4056, U8 DW01A, U9 TP4056, Y1 Crystal

Commit message: Final result
Parts:
- C25, R14, R20, R46, R54: moved to B.Cu
- C5, C6: footprint Capacitor_SMD:C_0805_2012Metric_Pad1.18x1.45mm_HandSolder -> Capacitor_SMD:C_0603_1608Metric_Pad1.08x0.95mm_HandSolder
- R10, R28, R29, R30, R31, R32, R35, R36, R37: footprint Resistor_SMD:R_1206_3216Metric_Pad1.30x1.75mm_HandSolder -> Capacitor_SMD:C_0805_2012Metric_Pad1.18x1.45mm_HandSolder
- R50: moved to F.Cu
- moved C22 103.6 mm to (106.0, 78.2)
- moved C23 103.6 mm to (108.0, 78.2), turned to -90 degrees
- moved R31 100.8 mm to (107.0, 73.8)
- moved R35 97.2 mm to (110.0, 86.2)
- moved R30 96.2 mm to (110.5, 72.5), turned to 180 degrees
- moved C24 92.1 mm to (106.2, 82.0), turned to 180 degrees
- moved C21 88.2 mm to (109.0, 63.8), turned to 0 degrees
- moved R29 87.9 mm to (108.6, 60.5), turned to 0 degrees
- moved R32 85.6 mm to (121.2, 85.2), turned to 180 degrees
- moved R37 81.8 mm to (110.2, 95.2)
- moved R28 81.6 mm to (112.5, 60.5), turned to 0 degrees
- moved R36 71.4 mm to (119.5, 98.2), turned to 180 degrees
- moved R16 63.1 mm to (113.8, 69.5)
- moved D2 62.9 mm to (113.8, 65.0)
- moved D3 62.9 mm to (116.8, 65.0)
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Connections:
- J5 pad SH: (no net) -> GND
- R20 pad 2: GATE_1 -> GATE_4
- R21 pad 2: GATE_2 -> GATE_3
- R22 pad 2: GATE_3 -> GATE_2
- R23 pad 2: GATE_4 -> GATE_1
- U4 pad 29: GATE_1 -> GATE_4
- U4 pad 30: GATE_2 -> GATE_3
- U4 pad 31: GATE_3 -> GATE_2
- U4 pad 32: GATE_4 -> GATE_1
- U4 pad 38: V_Sense1 -> V_Sense4
- U4 pad 39: V_Sense2 -> V_Sense3
- U4 pad 40: V_Sense3 -> V_Sense2
- U4 pad 41: V_Sense4 -> V_Sense1
Routing:
- net GND: track 109.7 -> 182.2 mm, vias 44 -> 68
- net Net-(U11-CE): track 0.00 -> 43.0 mm, vias 0 -> 1
- net V_Sense4: track 0.00 -> 38.6 mm, vias 0 -> 3
- net BAT+_2: track 0.00 -> 37.2 mm, vias 0 -> 1
- net BAT+_1: track 0.00 -> 36.0 mm, vias 0 -> 1
- net V_Sense3: track 0.00 -> 35.7 mm, vias 0 -> 3
- net Net-(U9-CE): track 0.00 -> 33.7 mm
- net Net-(U7-CE): track 0.00 -> 32.8 mm, vias 0 -> 1
- net Net-(U1-CE): track 0.00 -> 31.0 mm
- net V_Sense1: track 0.00 -> 29.1 mm
- net BAT+_4: track 0.00 -> 28.2 mm, vias 0 -> 1
- net BAT+_3: track 0.00 -> 25.7 mm, vias 0 -> 1
- net Net-(U9-~{CHRG}): track 0.00 -> 22.0 mm, vias 0 -> 1
- net V_Sense2: track 0.00 -> 21.7 mm
- net Net-(U1-~{STDBY}): track 0.00 -> 21.3 mm, vias 0 -> 1
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- added copper zone on In2.Cu, net +5V
- added copper zone on B.Cu, net GND
- added copper zone on In1.Cu, net GND
