File: PROJECT_1_V2.kicad_sch (KiCad schematic)
At the start: 125 parts, among them J1 Battery Input, J2 Battery Input, J3 Battery Input, J4 Battery Input, J5 USB_C_Receptacle_USB2.0_16P, Q10 DMG9926UDM, Q7 DMG9926UDM, Q8 DMG9926UDM, Q9 DMG9926UDM, SW1 RESET, SW2 BOOT_LOADER, U1 TP4056, U10 DW01A, U11 TP4056-42-ESOP8, U12 DW01A, U2 Nokia_5110_LCD, U3 LM2576T-3.3, U4 RP2040, U5 W25Q128JVS, U6 DW01A, U7 TP4056, U8 DW01A, U9 TP4056, Y1 Crystal

Commit message: Final result
Parts:
- C5, C6: footprint Capacitor_SMD:C_0805_2012Metric_Pad1.18x1.45mm_HandSolder -> Capacitor_SMD:C_0603_1608Metric_Pad1.08x0.95mm_HandSolder
- R10: footprint Resistor_SMD:R_1206_3216Metric_Pad1.30x1.75mm_HandSolder -> Capacitor_SMD:C_0805_2012Metric_Pad1.18x1.45mm_HandSolder
- R19: value 2k -> 1k
- R30: renamed from R43; value 2k -> 1k
- R37: renamed from R50; value 2k -> 1k
- R44: renamed from R57; value 2k -> 1k
- R45: renamed from R28; footprint Resistor_SMD:R_1206_3216Metric_Pad1.30x1.75mm_HandSolder -> Capacitor_SMD:C_0805_2012Metric_Pad1.18x1.45mm_HandSolder
- R46: renamed from R29; footprint Resistor_SMD:R_1206_3216Metric_Pad1.30x1.75mm_HandSolder -> Capacitor_SMD:C_0805_2012Metric_Pad1.18x1.45mm_HandSolder
- R47: renamed from R30; footprint Resistor_SMD:R_1206_3216Metric_Pad1.30x1.75mm_HandSolder -> Capacitor_SMD:C_0805_2012Metric_Pad1.18x1.45mm_HandSolder
- R48: renamed from R31; footprint Resistor_SMD:R_1206_3216Metric_Pad1.30x1.75mm_HandSolder -> Capacitor_SMD:C_0805_2012Metric_Pad1.18x1.45mm_HandSolder
- R49: renamed from R32; footprint Resistor_SMD:R_1206_3216Metric_Pad1.30x1.75mm_HandSolder -> Capacitor_SMD:C_0805_2012Metric_Pad1.18x1.45mm_HandSolder
- R50: renamed from R35; footprint Resistor_SMD:R_1206_3216Metric_Pad1.30x1.75mm_HandSolder -> Capacitor_SMD:C_0805_2012Metric_Pad1.18x1.45mm_HandSolder
- R51: renamed from R36; footprint Resistor_SMD:R_1206_3216Metric_Pad1.30x1.75mm_HandSolder -> Capacitor_SMD:C_0805_2012Metric_Pad1.18x1.45mm_HandSolder
- R52: renamed from R37; footprint Resistor_SMD:R_1206_3216Metric_Pad1.30x1.75mm_HandSolder -> Capacitor_SMD:C_0805_2012Metric_Pad1.18x1.45mm_HandSolder
- renumbered C25 to C21, C26 to C22, C27 to C23, C28 to C24, C29 to C25, C30 to C26, C31 to C27, C32 to C28, C33 to C29, C21 to C30, C22 to C31, C24 to C32, C23 to C33, R40 to R24, R39 to R25, R38 to R27, R41 to R28, R42 to R29, R47 to R31, R46 to R32, R44 to R33, R45 to R34, R48 to R35, R49 to R36, R54 to R38, R53 to R39, R51 to R40, R52 to R41, R55 to R42, R56 to R43, R33 to R53, R34 to R54
Connections:
- net GATE_1: now also R23.2, U4.32 (GPIO21); no longer R20.2, U4.29 (GPIO18)
- net GATE_2: now also R22.2, U4.31 (GPIO20); no longer R21.2, U4.30 (GPIO19)
- net GATE_3: now also R21.2, U4.30 (GPIO19); no longer R22.2, U4.31 (GPIO20)
- net GATE_4: now also R20.2, U4.29 (GPIO18); no longer R23.2, U4.32 (GPIO21)
- net V_Sense1: now also U4.41 (GPIO29/ADC3); no longer U4.38 (GPIO26/ADC0)
- net V_Sense2: now also U4.40 (GPIO28/ADC2); no longer U4.39 (GPIO27/ADC1)
- net V_Sense3: now also U4.39 (GPIO27/ADC1); no longer U4.40 (GPIO28/ADC2)
- net V_Sense4: now also U4.38 (GPIO26/ADC0); no longer U4.41 (GPIO29/ADC3)
- no-connect marks 24 -> 23
